File: processor_CM5.kicad_sch (KiCad schematic)
At the start: 0 parts

Commit message: added MAX177330 CHG
Parts:
- added U1: CM5104032, symbol DIY Pi Smartphone Library:CM5104032
Connections:
- new net SCL: U1.56 (GPIO3)
- new net SDA: U1.58 (GPIO2)
